File: Hardware/1000026_V0b/1000026_V0b.kicad_pcb (KiCad board)
At the start: 4 copper layers, 100 x 70 mm, 29 parts, among them J1 MOLEX_533750410, J2 4390, J3 532580229, J5 532580229, J9 0525591853, SW1 SW4_TL3305CF260QG_EWI, U1 TO252-3_ROM, U2 MAX7480ESA+

Commit message: Updating SW and PCB 1000026
Parts:
- C1: value CAPC3216X94N -> 12065C503JAT2A
- C2, C3: value CAPC3325X127N -> 12102C104KAT2A
- C4: value CAP_CL32_SAM -> CL32B475KBUYNNE
- C5: value CAP_CL32_SAM -> CL32A106KAULNNE
- D2: value DO-41_DIO -> 1N4007G-T
- D5: value SOD123_DIO -> BZT52C3V3-7-F
- J1: value MOLEX_533750410 -> 533750410
- LED1, LED2: value SMD-2_3P2X1P7_ONS -> QTLP650D4TR
- S1: value Slider_switch_500SSP1S2M2QEA -> 500SSP1S2M2QEA
- SW1: value SW4_TL3305CF260QG_EWI -> TL3305CF260QG
- U1: value TO252-3_ROM -> BD450M5FP-CE2
Connections:
- A1 pad 21: bit_2 -> bit_0
- A1 pad 26: bit_0 -> bit_2
Routing:
- net 7.4V: track 198.3 -> 171.0 mm
- net unconnected-(S1-Pad2): track 0.00 -> 18.2 mm
- net GND: track 175.3 -> 184.3 mm
Changed lines of the file:
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@@
       (effects (font (size 1 1) (thickness 0.2)))
     )
-    (fp_text value "SMD-2_3P2X1P7_ONS" (at 0.2286 4.6228 unlocked) (layer "F.Fab") hide
+    (fp_text value "QTLP650D4TR" (at 0.2286 4.6228 unlocked) (layer "F.Fab") hide
       (effects (font (size 1 1) (thickness 0.2)))
     )
@@
       (effects (font (size 1 1) (thickness 0.2)))
     )
-    (fp_text value "CAP_CL32_SAM" (at 0.2032 9.525 -90 unlocked) (layer "F.Fab") hide
+    (fp_text value "CL32A106KAULNNE" (at 0.2032 9.525 -90 unlocked) (layer "F.Fab") hide
       (effects (font (size 1 1) (thickness 0.2)))
     )
@@
       (effects (font (size 1 1) (thickness 0.2)))
     )
-    (fp_text value "CAPC3325X127N" (at 0.2286 2.3876 -90) (layer "F.Fab") hide
+    (fp_text value "12102C104KAT2A" (at 0.2286 2.3876 -90) (layer "F.Fab") hide
       (effects (font (size 1 1) (thickness 0.2)))
     )
@@
       (effects (font (size 1 1) (thickness 0.2)))
     )
-    (fp_text value "CAPC3325X127N" (at 0.2286 2.3876 -90) (layer "F.Fab") hide
+    (fp_text value "12102C104KAT2A" (at 0.2286 2.3876 -90) (layer "F.Fab") hide
       (effects (font (size 1 1) (thickness 0.2)))
     )
@@
       (effects (font (size 1 1) (thickness 0.2)))
     )
-    (fp_text value "CAP_CL32_SAM" (at 0 6.858 -90 unlocked) (layer "F.Fab") hide
+    (fp_text value "CL32B475KBUYNNE" (at 0 6.858 -90 unlocked) (layer "F.Fab") hide
       (effects (font (size 1 1) (thickness 0.2)))
     )
@@
       (effects (font (size 1 1) (thickness 0.2)))
     )
-    (fp_text value "SOD123_DIO" (at -0.5 2.75 -90 unlocked) (layer "F.Fab") hide
+    (fp_text value "BZT52C3V3-7-F" (at -0.5 2.75 -90 unlocked) (layer "F.Fab") hide
       (effects (font (size 1 1) (thickness 0.2)))
     )
@@
       (effects (font (size 1 1) (thickness 0.2)))
     )
-    (fp_text value "SW4_TL3305CF260QG_EWI" (at -0.1016 5.588 unlocked) (layer "F.Fab") hide
+    (fp_text value "TL3305CF260QG" (at -0.1016 5.588 unlocked) (layer "F.Fab") hide
       (effects (font (size 1 1) (thickness 0.2)))
     )
@@
       (net 41 "HREF") (pinfunction "D15/A1") (pintype "bidirectional"))
     (pad "21" thru_hole oval (at 15.24 22.86 180) (size 1.6 1.6) (drill 1) (layers *.Cu *.Mask)
-      (net 21 "bit_2") (pinfunction "D16/A2") (pintype "bidirectional"))
+      (net 19 "bit_0") (pinfunction "D16/A2") (pintype "bidirectional"))
     (pad "22" thru_hole oval (at 15.24 20.32 180) (size 1.6 1.6) (drill 1) (layers *.Cu *.Mask)
       (net 32 "PB") (pinfunction "D17/A3") (pintype "bidirectional"))
@@
       (net 20 "bit_1") (pinfunction "D20/A6") (pintype "bidirectional"))
     (pad "26" thru_hole oval (at 15.24 10.16 180) (size 1.6 1.6) (drill 1) (layers *.Cu *.Mask)
-      (net 19 "bit_0") (pinfunction "D21/A7") (pintype "bidirectional"))
+      (net 21 "bit_2") (pinfunction "D21/A7") (pintype "bidirectional"))
     (pad "27" thru_hole oval (at 15.24 7.62 180) (size 1.6 1.6) (drill 1) (layers *.Cu *.Mask)
       (net 53 "unconnected-(A1-Pad27)") (pinfunction "+5V") (pintype "power_out+no_connect"))
@@
       (effects (font (size 1 1) (thickness 0.2)))
     )
-    (fp_text value "SMD-2_3P2X1P7_ONS" (at 0.2286 4.6228 180 unlocked) (layer "F.Fab") hide
+    (fp_text value "QTLP650D4TR" (at 0.2286 4.6228 180 unlocked) (layer "F.Fab") hide
       (effects (font (size 1 1) (thickness 0.2)))
     )
@@
       (effects (font (size 1 1) (thickness 0.2)))
     )
-    (fp_text value "MOLEX_533750410" (at -3.048 10.4394 -90) (layer "F.Fab") hide
+    (fp_text value "533750410" (at -3.048 10.4394 -90) (layer "F.Fab") hide
       (effects (font (size 1 1) (thickness 0.2)))
     )
@@
       (effects (font (size 1 1) (thickness 0.2)))
     )
-    (fp_text value "Slider_switch_500SSP1S2M2QEA" (at 0 8.128 180) (layer "F.Fab") hide
+    (fp_text value "500SSP1S2M2QEA" (at 0 8.128 180) (layer "F.Fab") hide
       (effects (font (size 1 1) (thickness 0.2)))
     )
@@
       (effects (font (size 1 1) (thickness 0.2)))
     )
-    (fp_text value "CAPC3216X94N" (at 0.2032 2.3368 -90) (layer "F.Fab") hide
+    (fp_text value "12065C503JAT2A" (at 0.2032 2.3368 -90) (layer "F.Fab") hide
       (effects (font (size 1 1) (thickness 0.2)))
     )
@@
       (effects (font (size 1 1) (thickness 0.2)))
     )
-    (fp_text value "TO252-3_ROM" (at 0.1016 11.9634 unlocked) (layer "F.Fab") hide
+    (fp_text value "BD450M5FP-CE2" (at 0.1016 11.9634 unlocked) (layer "F.Fab") hide
       (effects (font (size 1 1) (thickness 0.2)))
     )
@@
       (effects (font (size 1 1) (thickness 0.2)))
     )
-    (fp_text value "DO-41_DIO" (at 5.238 -3.42125 unlocked) (layer "F.Fab") hide
+    (fp_text value "1N4007G-T" (at 5.238 -3.42125 unlocked) (layer "F.Fab") hide
       (effects (font (size 1 1) (thickness 0.2)))
     )
@@
   (segment (start 102.3648 93.2882) (end 102.3648 93.1382) (width 0.25) (layer "F.Cu") (net 37))
   (segment (start 144.0876 117.8965) (end 144.0876 120.011) (width 0.25) (layer "F.Cu") (net 37))
+  (segment (start 118.3876 69.1132) (end 118.3876 73.5334) (width 0.25) (layer "F.Cu") (net 37))
+  (segment (start 118.3876 73.5334) (end 115.1078 76.8132) (width 0.25) (layer "F.Cu") (net 37))
   (segment (start 106.854799 68.038191) (end 114.416991 68.038191) (width 0.25) (layer "F.Cu") (net 37))
   (segment (start 121.8769 93.1382) (end 123.9119 95.1732) (width 0.25) (layer "F.Cu") (net 37))
@@
   (segment (start 144.6398 99.263197) (end 146.6148 97.288197) (width 0.25) (layer "F.Cu") (net 40))
   (segment (start 144.6398 100.2632) (end 144.4398 100.4632) (width 0.25) (layer "F.Cu") (net 40))
-  (segment (start 118.3876 69.1132) (end 118.3876 73.5334) (width 0.25) (layer "F.Cu") (net 40))
   (segment (start 139.0398 109.2632) (end 141.7398 106.5632) (width 0.25) (layer "F.Cu") (net 40))
-  (segment (start 118.3876 73.5334) (end 115.1078 76.8132) (width 0.25) (layer "F.Cu") (net 40))
   (segment (start 141.192 117.7632) (end 141.192 117.8965) (width 0.25) (layer "F.Cu") (net 40))
   (segment (start 140.666426 111.855826) (end 141.3238 112.5132) (width 0.25) (layer "F.Cu") (net 40))
@@
   (segment (start 119.71105 57.53445) (end 118.5778 57.53445) (width 0.25) (layer "In1.Cu") (net 40))
   (segment (start 127.5898 109.7132) (end 127.5898 114.110226) (width 0.25) (layer "In1.Cu") (net 40))
-  (segment (start 117.242764 108.46319) (end 122.8898 114.110226) (width 0.25) (layer "In1.Cu") (net 40))
-  (segment (start 106.979799 108.46319) (end 117.242764 108.46319) (width 0.25) (layer "In1.Cu") (net 40))
   (segment (start 127.5898 109.7132) (end 116.4898 98.6132) (width 0.25) (layer "In1.Cu") (net 40))
   (segment (start 107.4018 63.991189) (end 106.854799 64.53819) (width 0.25) (layer "In1.Cu") (net 40))
@@
   (segment (start 155.5148 96.513199) (end 156.4898 97.488199) (width 0.25) (layer "F.Cu") (net 59))
   (segment (start 154.439801 96.513199) (end 155.5148 96.513199) (width 0.25) (layer "F.Cu") (net 59))
+  (segment (start 117.242764 108.46319) (end 122.8898 114.110226) (width 0.25) (layer "In1.Cu") (net 61))
+  (segment (start 106.979799 108.46319) (end 117.242764 108.46319) (width 0.25) (layer "In1.Cu") (net 61))
 )

Commit message: updating a file.
Other:
- board text added: "user pushbutton"
- board text removed: "->reset->ready"
Changed lines of the file:
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@@
-      (effects (font (size 1 1) (thickness 0.2)))
-    )
-    (fp_text user "motion control<-" (at 7.0121 -6.625 180) (layer "F.SilkS")
       (effects (font (size 1 1) (thickness 0.2)))
     )
@@
       (effects (font (size 1 1) (thickness 0.2)))
     )
-    (fp_text user "<-motion commands" (at 7.125 -6.325 180) (layer "F.SilkS")
-      (effects (font (size 1 1) (thickness 0.2)))
-    )
     (fp_text user "USB" (at 7.62 35.56 180 unlocked) (layer "F.SilkS")
       (effects (font (size 1 1) (thickness 0.2)))
@@
     (effects (font (size 1 1) (thickness 0.2)))
   )
-  (gr_text "->reset->ready" (at 177.1898 117.3132) (layer "F.SilkS")
+  (gr_text "user pushbutton" (at 177.1898 117.3132) (layer "F.SilkS")
     (effects (font (size 1 1) (thickness 0.2)))
   )
