File: Hardware/1000026_V0b/1000026_V0b.kicad_sch (KiCad schematic)
At the start: 29 parts, among them J1 533750410, J2 4390, J3 532580229, J5 532580229, J9 0525591853, SW1 TL3305CF260QG, U1 BD450M5FP-CE2, U2 MAX7480ESA+

Commit message: Updating SW and PCB 1000026
Connections:
- net bit_0: now also A1.21 (D16/A2); no longer A1.26 (D21/A7)
- net bit_2: now also A1.26 (D21/A7); no longer A1.21 (D16/A2)
Changed lines of the file:
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@@
     )
   )
-  (global_label "bit_0" (shape input) (at 173.736 70.866 180) (fields_autoplaced)
+  (global_label "bit_2" (shape input) (at 173.736 70.866 180) (fields_autoplaced)
     (effects (font (size 1.27 1.27)) (justify right))
     (property "Intersheet References" "${INTERSHEET_REFS}" (id 0) (at 166.6662 70.7866 0)
@@
     )
   )
-  (global_label "bit_2" (shape input) (at 183.388 58.166 180) (fields_autoplaced)
+  (global_label "bit_0" (shape input) (at 183.388 58.166 180) (fields_autoplaced)
     (effects (font (size 1.27 1.27)) (justify right))
     (property "Intersheet References" "${INTERSHEET_REFS}" (id 0) (at 176.3182 58.0866 0)

Commit message: Updating SW, digital ok
Connections:
- net bit_0: now also A2.12 (~D9); no longer A2.10 (D7)
- net bit_2: now also A2.10 (D7); no longer A2.12 (~D9)
Changed lines of the file:
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@@
     (stroke (width 0) (type default) (color 0 0 0 0))
   )
-  (wire (pts (xy 137.16 54.356) (xy 149.3774 54.1528))
+  (wire (pts (xy 137.16 54.356) (xy 149.352 54.356))
     (stroke (width 0) (type default) (color 0 0 0 0))
   )
@@
     )
   )
-  (global_label "bit_1" (shape input) (at 149.3774 54.1528 0) (fields_autoplaced)
-    (effects (font (size 1.27 1.27)) (justify left))
-    (property "Intersheet References" "${INTERSHEET_REFS}" (id 0) (at 156.4472 54.0734 0)
+  (global_label "bit_1" (shape input) (at 149.352 54.356 0) (fields_autoplaced)
+    (effects (font (size 1.27 1.27)) (justify left))
+    (property "Intersheet References" "${INTERSHEET_REFS}" (id 0) (at 156.4218 54.2766 0)
       (effects (font (size 1.27 1.27)) (justify left) hide)
     )
@@
     )
   )
-  (global_label "bit_2" (shape input) (at 139.446 51.816 0) (fields_autoplaced)
+  (global_label "bit_0" (shape input) (at 139.446 51.816 0) (fields_autoplaced)
     (effects (font (size 1.27 1.27)) (justify left))
     (property "Intersheet References" "${INTERSHEET_REFS}" (id 0) (at 146.5158 51.7366 0)
@@
     )
   )
-  (global_label "bit_0" (shape input) (at 139.446 56.896 0) (fields_autoplaced)
+  (global_label "bit_2" (shape input) (at 139.446 56.896 0) (fields_autoplaced)
     (effects (font (size 1.27 1.27)) (justify left))
     (property "Intersheet References" "${INTERSHEET_REFS}" (id 0) (at 146.5158 56.8166 0)
